Commit message: update English annotations

File: ws_robot_arm/src/model/xacro/model/base_footlink.xacro (robot description, xacro)
@@ -1,4 +1,4 @@
 <robot name="arm_dyn" xmlns:xacro="http://wiki.ros.org/xacro">
-    <!-- 机械臂参数 -->
+    <!-- Mechanical arm parameters -->
     <xacro:property name="pi" value="3.14159265358979" />
     <xacro:property name="joint_lower" value="${-pi}" />
@@ -11,11 +11,11 @@
     <xacro:property name="fixed_block_length" value="2" />
     <xacro:property name="fixed_block_wide" value="2" />
-    <!-- 建立基点连杆 -->
+    <!-- create a base link -->
     <link name="base_footlink">
-        <!-- 可视化 -->
+        <!-- visualization -->
         <visual>
-            <!-- 外观 -->
+            <!-- appearance -->
             <geometry>
-                <sphere radius="0.00001" />   <!-- 球体 -->
+                <sphere radius="0.00001" />   <!-- sphere -->
             </geometry>
         </visual>
@@ -29,21 +29,21 @@
        </inertial>
    </xacro:macro>
-    <!-- 固定块 -->
+    <!-- Fixed block -->
     <link name="fixed_block_link">
-        <!-- 可视化 -->
+        <!-- visualization -->
         <visual>
-            <!-- 外观 -->
+            <!-- appearance -->
             <geometry>
-                <box size="${fixed_block_length} ${fixed_block_wide} ${fixed_block_high}" />   <!-- 导入外部模型 -->
+                <box size="${fixed_block_length} ${fixed_block_wide} ${fixed_block_high}" />   <!-- Import external models -->
             </geometry>
-            <origin xyz="0 0 0" rpy="0 0 0" />    <!-- 连杆偏移量 -->
-            <!-- 材质 -->
+            <origin xyz="0 0 0" rpy="0 0 0" />    <!-- Linkage offset -->
+            <!-- texture of material -->
             <material name="">
-                <color rgba="0.8 0.8 0.8 1" />    <!-- 颜色 -->
+                <color rgba="0.8 0.8 0.8 1" />    <!-- colour -->
             </material>
         </visual>
-        <!-- 碰撞矩阵 -->
+        <!-- Collision matrix -->
         <collision>
-            <!-- 外观 -->
+            <!-- appearance -->
             <geometry>
                 <box size="${fixed_block_length} ${fixed_block_wide} ${fixed_block_high}" />
@@ -51,12 +51,12 @@
             <origin xyz="0 0 0" rpy="0 0 0" />
         </collision>
-        <!-- 惯性矩阵 -->
+        <!-- Inertia matrix -->
         <xacro:Box_inertial_matrix m="1000" l="${fixed_block_length}" w="${fixed_block_wide}" h="${fixed_block_high}" />
     </link>
-    <!-- 建立固定块与位置基点的连接关节 -->
-    <joint name="fixed_block_joint" type="fixed"> <!-- 关节标签 -->
-        <parent link="base_footlink" /> <!-- 父级标签 -->
-        <child link="fixed_block_link" /> <!-- 子级标签 -->
-        <origin xyz="0 0 ${fixed_block_high/2}" rpy="0 0 0" /> <!-- 偏移量标签 -->
+    <!-- Establish a connection joint between a fixed block and a positional base point -->
+    <joint name="fixed_block_joint" type="fixed">
+        <parent link="base_footlink" />
+        <child link="fixed_block_link" />
+        <origin xyz="0 0 ${fixed_block_high/2}" rpy="0 0 0" />
     </joint>
     <gazebo reference="fixed_block_link">

File: ws_robot_arm/src/model/xacro/model/base_link.xacro (robot description, xacro)
@@ -1,19 +1,14 @@
 <robot name="arm_dyn" xmlns:xacro="http://wiki.ros.org/xacro">
-    <!-- 创建基座连杆 -->
     <xacro:macro name="Base_link_create" params="name pos_l pos_w">
-        <link name="${name}">     <!-- 连杆 -->
-            <!-- 可视化 -->
+        <link name="${name}">
             <visual>
-                <!-- 外观 -->
                 <geometry>
-                    <mesh filename="package://model/meshes/base_link.STL" />   <!-- 导入外部模型 -->
+                    <mesh filename="package://model/meshes/base_link.STL" />
                 </geometry>
-                <origin xyz="0 0 0" rpy="0 0 0" />    <!-- 连杆偏移量 -->
-                <!-- 材质 -->
+                <origin xyz="0 0 0" rpy="0 0 0" />
                 <material name="">
-                    <color rgba="0.4 0.4 0.4 1" />    <!-- 颜色 -->
+                    <color rgba="0.4 0.4 0.4 1" />
                 </material>
             </visual>
-            <!-- 碰撞矩阵 -->
             <collision>
                 <geometry>
@@ -22,5 +17,4 @@
                 <origin xyz="0 0 0" rpy="0 0 0" />
             </collision>
-            <!-- 惯性矩阵 -->
             <inertial>
                 <origin xyz="2.0867E-05 0.0024582 0.036484" rpy="0 0 0" />
@@ -29,9 +23,8 @@
             </inertial>
         </link>
-        <!-- 建立底座与位置基点的连接关节 -->
-        <joint name="${name}_joint" type="fixed"> <!-- 关节标签 -->
-            <parent link="fixed_block_link" /> <!-- 父级标签 -->
-            <child link="${name}" /> <!-- 子级标签 -->
-            <origin xyz="${pos_l} ${pos_w} ${fixed_block_high/2}" rpy="0 0 0" /> <!-- 偏移量标签 -->
+        <joint name="${name}_joint" type="fixed">
+            <parent link="fixed_block_link" />
+            <child link="${name}" />
+            <origin xyz="${pos_l} ${pos_w} ${fixed_block_high/2}" rpy="0 0 0" />
         </joint>
         <gazebo reference="${name}">

File: ws_robot_arm/src/model/xacro/model/link1.xacro (robot description, xacro)
@@ -1,5 +1,4 @@
 <robot name="arm_dyn" xmlns:xacro="http://wiki.ros.org/xacro">
     <xacro:macro name="Link1_create" params="name joint_parent">
-        <!-- 连杆1 -->
         <link name="${name}">
             <visual>

File: ws_robot_arm/src/model/xacro/model/link2.xacro (robot description, xacro)
@@ -1,5 +1,4 @@
 <robot name="arm_dyn" xmlns:xacro="http://wiki.ros.org/xacro">
   <xacro:macro name="Link2_create" params="name joint_parent">
-    <!-- 连杆2 -->
     <link name="${name}">
       <visual>

File: ws_robot_arm/src/model/xacro/model/link3.xacro (robot description, xacro)
@@ -1,5 +1,4 @@
 <robot name="arm_dyn" xmlns:xacro="http://wiki.ros.org/xacro">
   <xacro:macro name="Link3_create" params="name joint_parent">
-    <!-- 连杆3 -->
     <link name="${name}">
       <inertial>

File: ws_robot_arm/src/model/xacro/model/link4.xacro (robot description, xacro)
@@ -1,5 +1,4 @@
 <robot name="arm_dyn" xmlns:xacro="http://wiki.ros.org/xacro">
   <xacro:macro name="Link4_create" params="name joint_parent">
-      <!-- 连杆4 -->
     <link name="${name}">
       <visual>

File: ws_robot_arm/src/model/xacro/model/link5.xacro (robot description, xacro)
@@ -1,5 +1,4 @@
 <robot name="arm_dyn" xmlns:xacro="http://wiki.ros.org/xacro">
   <xacro:macro name="Link5_create" params="name joint_parent">
-      <!-- 连杆5 -->
     <link name="${name}">
       <visual>

File: ws_robot_arm/src/model/xacro/model/my_arm.xacro (robot description, xacro)
@@ -1,4 +1,3 @@
 <robot name="arm_dyn" xmlns:xacro="http://wiki.ros.org/xacro">
-    <!-- 包括文件 -->
     <xacro:include filename="base_footlink.xacro" />
     <xacro:include filename="base_link.xacro" />
@@ -11,5 +10,5 @@
     <xacro:include filename="link7.xacro" />
     <xacro:include filename="tran.xacro" />
-    <!-- 创建一台机械臂 -->
+    <!-- Create a robotic arm -->
     <xacro:macro name="Robot_arm_create" params="arm_number pos_l pos_w">
         <xacro:Base_link_create name="base_link${arm_number}" pos_l="${pos_l}" pos_w="${pos_w}" />
@@ -30,5 +29,4 @@
         <xacro:joint_transmission joint_name="link${arm_number}_7_joint" />
     </xacro:macro>
-    <!-- 创建机械臂 -->
     <xacro:Robot_arm_create arm_number="1" pos_l="-${fixed_block_length/2-0.5}" pos_w="${fixed_block_wide/2-0.5}" />
     <xacro:Robot_arm_create arm_number="2" pos_l="-${fixed_block_length/2-0.5}" pos_w="-${fixed_block_wide/2-0.5}" />

Commit message: common update

File: ws_robot_arm/src/model/xacro/model/base_footlink.xacro (robot description, xacro)
@@ -11,14 +11,4 @@
     <xacro:property name="fixed_block_length" value="2" />
     <xacro:property name="fixed_block_wide" value="2" />
-    <!-- create a base link -->
-    <link name="base_footlink">
-        <!-- visualization -->
-        <visual>
-            <!-- appearance -->
-            <geometry>
-                <sphere radius="0.00001" />   <!-- sphere -->
-            </geometry>
-        </visual>
-    </link>
     <xacro:macro name="Box_inertial_matrix" params="m l w h">
        <inertial>
@@ -54,10 +44,4 @@
         <xacro:Box_inertial_matrix m="1000" l="${fixed_block_length}" w="${fixed_block_wide}" h="${fixed_block_high}" />
     </link>
-    <!-- Establish a connection joint between a fixed block and a positional base point -->
-    <joint name="fixed_block_joint" type="fixed">
-        <parent link="base_footlink" />
-        <child link="fixed_block_link" />
-        <origin xyz="0 0 ${fixed_block_high/2}" rpy="0 0 0" />
-    </joint>
     <gazebo reference="fixed_block_link">
         <material>Gazebo/Grey</material>

File: ws_robot_arm/src/model/xacro/model/my_arm.xacro (robot description, xacro)
@@ -30,4 +30,4 @@
     </xacro:macro>
     <xacro:Robot_arm_create arm_number="1" pos_l="-${fixed_block_length/2-0.5}" pos_w="${fixed_block_wide/2-0.5}" />
-    <xacro:Robot_arm_create arm_number="2" pos_l="-${fixed_block_length/2-0.5}" pos_w="-${fixed_block_wide/2-0.5}" />
+    <!-- <xacro:Robot_arm_create arm_number="2" pos_l="-${fixed_block_length/2-0.5}" pos_w="-${fixed_block_wide/2-0.5}" /> -->
 </robot>
